File: hw/podlewaczka.kicad_pcb (KiCad board)
At the start: 2 copper layers, 59 parts, among them J1 UART, J10 Screw_Terminal_01x01, J11 Screw_Terminal_01x01, J12 Ext IO, J2 Solar panel input, J3 Battery input, J4 I2C Sensor connector, J5 Pump3, J6 Pump1, J7 Pump2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

Commit message: PCB update
Parts:
- moved R23 60.1 mm to (125.8, 99.0), turned to 90 degrees
- moved Q4 58.3 mm to (128.5, 97.2)
- moved R22 57.0 mm to (128.5, 94.5)
- moved Q5 54.3 mm to (128.5, 100.9)
Routing:
- net Net-(Q5-Pad3): track 13.2 -> 39.9 mm, vias 0 -> 2
- net /RTS: track 0.00 -> 19.9 mm, vias 0 -> 1
- net Net-(D4-Pad1): track 0.00 -> 12.0 mm
- net /DTR: track 0.00 -> 11.7 mm, vias 0 -> 1
- net Net-(J12-Pad2): track 37.9 -> 46.2 mm, vias 0 -> 2
- net Net-(D1-Pad1): track 7.01 -> 13.7 mm
- net Net-(R14-Pad2): track 41.3 -> 47.9 mm
- net Net-(D5-Pad1): track 0.00 -> 6.29 mm
- net VCC: track 38.4 -> 42.0 mm
- net Net-(Q1-Pad1): track 0.00 -> 1.83 mm
- net Net-(Q4-Pad1): track 0.00 -> 1.80 mm
- net Net-(Q5-Pad1): track 0.00 -> 1.73 mm

Commit message: Finished PCB
Routing:
- net GND: vias 0 -> 72
- added copper zone on B.Cu, net GND
- added copper zone on F.Cu, net GND
Other:
- board text added: "Garden monitoring system v1.0"
Changed lines of the file:
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@@
-(kicad_pcb (version 20171130) (host pcbnew "(5.0.0)")
+(kicad_pcb (version 20171130) (host pcbnew 5.0.0-fee4fd1~66~ubuntu18.04.1)
   (general
     (thickness 1.6)
-    (drawings 20)
-    (tracks 393)
+    (drawings 21)
+    (tracks 467)
     (zones 0)
     (modules 59)
@@
     (visible_elements 7FFFFFFF)
     (pcbplotparams
-      (layerselection 0x010fc_ffffffff)
+      (layerselection 0x020f0_ffffffff)
       (usegerberextensions false)
       (usegerberattributes false)
@@
       (outputformat 1)
       (mirror false)
-      (drillshape 1)
+      (drillshape 0)
       (scaleselection 1)
-      (outputdirectory ""))
+      (outputdirectory "output/"))
   )
   (net 0 "")
@@
     )
   )
+  (gr_text "Garden\nmonitoring\nsystem v1.0" (at 139.75 84) (layer F.SilkS)
+    (effects (font (size 1.5 1.5) (thickness 0.3)))
+  )
   (gr_text GND (at 121.5 109.65) (layer F.SilkS)
     (effects (font (size 1 1) (thickness 0.15)))
@@
   (gr_line (start 175 55) (end 175 121) (layer Margin) (width 0.2))
   (gr_line (start 115 55) (end 175 55) (layer Margin) (width 0.2))
+  (via (at 158.75 98.75) (size 0.7) (drill 0.3) (layers F.Cu B.Cu) (net 2))
+  (via (at 160.25 79.5) (size 0.7) (drill 0.3) (layers F.Cu B.Cu) (net 2))
+  (via (at 159 79.5) (size 0.7) (drill 0.3) (layers F.Cu B.Cu) (net 2))
+  (via (at 160.25 78.25) (size 0.7) (drill 0.3) (layers F.Cu B.Cu) (net 2))
+  (via (at 159 78.25) (size 0.7) (drill 0.3) (layers F.Cu B.Cu) (net 2))
   (via (at 155.6 104.2) (size 0.7) (drill 0.3) (layers F.Cu B.Cu) (net 1))
   (via (at 155.6 113) (size 0.7) (drill 0.3) (layers F.Cu B.Cu) (net 1))
@@
   (segment (start 119.41 94.91) (end 118 94.91) (width 0.8) (layer F.Cu) (net 1))
   (segment (start 120.5 96) (end 119.41 94.91) (width 0.8) (layer F.Cu) (net 1))
-  (segment (start 157.5 95.25) (end 157.5 98.2625) (width 0.5) (layer F.Cu) (net 2))
+  (segment (start 157.5 95.25) (end 157.5 97.25) (width 0.5) (layer F.Cu) (net 2))
   (segment (start 156.4 95.25) (end 157.5 95.25) (width 0.5) (layer F.Cu) (net 2))
-  (segment (start 159.9875 94.5125) (end 161.5 94.5125) (width 0.5) (layer F.Cu) (net 2))
+  (segment (start 159.9875 94.5125) (end 160.25 94.5125) (width 0.5) (layer F.Cu) (net 2))
   (segment (start 159.25 95.25) (end 159.9875 94.5125) (width 0.5) (layer F.Cu) (net 2))
   (segment (start 157.5 95.25) (end 159.25 95.25) (width 0.5) (layer F.Cu) (net 2))
+  (via (at 157.75 78.25) (size 0.7) (drill 0.3) (layers F.Cu B.Cu) (net 2))
+  (via (at 157.75 79.5) (size 0.7) (drill 0.3) (layers F.Cu B.Cu) (net 2))
+  (via (at 161.5 79.5) (size 0.7) (drill 0.3) (layers F.Cu B.Cu) (net 2))
+  (via (at 161.5 78.25) (size 0.7) (drill 0.3) (layers F.Cu B.Cu) (net 2))
+  (via (at 137.25 120.25) (size 0.7) (drill 0.3) (layers F.Cu B.Cu) (net 2))
+  (via (at 139.5 120.25) (size 0.7) (drill 0.3) (layers F.Cu B.Cu) (net 2))
+  (via (at 142 120.25) (size 0.7) (drill 0.3) (layers F.Cu B.Cu) (net 2))
+  (via (at 144.75 120.25) (size 0.7) (drill 0.3) (layers F.Cu B.Cu) (net 2))
+  (via (at 147 120.25) (size 0.7) (drill 0.3) (layers F.Cu B.Cu) (net 2))
+  (via (at 138.5 113.75) (size 0.7) (drill 0.3) (layers F.Cu B.Cu) (net 2))
+  (via (at 144.75 117) (size 0.7) (drill 0.3) (layers F.Cu B.Cu) (net 2))
+  (via (at 140.25 107.75) (size 0.7) (drill 0.3) (layers F.Cu B.Cu) (net 2))
+  (via (at 146.75 110.75) (size 0.7) (drill 0.3) (layers F.Cu B.Cu) (net 2))
+  (via (at 143.75 101.75) (size 0.7) (drill 0.3) (layers F.Cu B.Cu) (net 2))
+  (via (at 138.75 101.75) (size 0.7) (drill 0.3) (layers F.Cu B.Cu) (net 2))
+  (via (at 135.25 101.75) (size 0.7) (drill 0.3) (layers F.Cu B.Cu) (net 2))
+  (via (at 131.5 106.25) (size 0.7) (drill 0.3) (layers F.Cu B.Cu) (net 2))
+  (via (at 134.5 104.75) (size 0.7) (drill 0.3) (layers F.Cu B.Cu) (net 2))
+  (via (at 127.25 103.25) (size 0.7) (drill 0.3) (layers F.Cu B.Cu) (net 2))
+  (via (at 126.25 114) (size 0.7) (drill 0.3) (layers F.Cu B.Cu) (net 2))
+  (via (at 128.25 115.75) (size 0.7) (drill 0.3) (layers F.Cu B.Cu) (net 2))
+  (via (at 160.5 120.25) (size 0.7) (drill 0.3) (layers F.Cu B.Cu) (net 2))
+  (via (at 157.25 109) (size 0.7) (drill 0.3) (layers F.Cu B.Cu) (net 2))
+  (via (at 154 109.25) (size 0.7) (drill 0.3) (layers F.Cu B.Cu) (net 2))
+  (via (at 156 98.75) (size 0.7) (drill 0.3) (layers F.Cu B.Cu) (net 2))
+  (segment (start 157.5 97.25) (end 157.5 98.2625) (width 0.5) (layer F.Cu) (net 2))
+  (via (at 157.5 97.25) (size 0.7) (drill 0.3) (layers F.Cu B.Cu) (net 2))
+  (via (at 154.75 95.5) (size 0.7) (drill 0.3) (layers F.Cu B.Cu) (net 2))
+  (segment (start 160.25 94.5125) (end 161.5 94.5125) (width 0.5) (layer F.Cu) (net 2))
+  (via (at 160.25 94.5125) (size 0.7) (drill 0.3) (layers F.Cu B.Cu) (net 2))
+  (via (at 163.75 94.5) (size 0.7) (drill 0.3) (layers F.Cu B.Cu) (net 2))
+  (via (at 165.5 94.5) (size 0.7) (drill 0.3) (layers F.Cu B.Cu) (net 2))
+  (via (at 148.25 97) (size 0.7) (drill 0.3) (layers F.Cu B.Cu) (net 2))
+  (via (at 142.25 94.75) (size 0.7) (drill 0.3) (layers F.Cu B.Cu) (net 2))
+  (via (at 150.75 90.75) (size 0.7) (drill 0.3) (layers F.Cu B.Cu) (net 2))
+  (via (at 150 83.75) (size 0.7) (drill 0.3) (layers F.Cu B.Cu) (net 2))
+  (via (at 144 76.5) (size 0.7) (drill 0.3) (layers F.Cu B.Cu) (net 2))
+  (via (at 134 78.25) (size 0.7) (drill 0.3) (layers F.Cu B.Cu) (net 2))
+  (via (at 140.5 81) (size 0.7) (drill 0.3) (layers F.Cu B.Cu) (net 2))
+  (via (at 129.75 83.25) (size 0.7) (drill 0.3) (layers F.Cu B.Cu) (net 2))
+  (via (at 134.75 83.5) (size 0.7) (drill 0.3) (layers F.Cu B.Cu) (net 2))
+  (via (at 138.5 86.5) (size 0.7) (drill 0.3) (layers F.Cu B.Cu) (net 2))
+  (via (at 124.25 90.5) (size 0.7) (drill 0.3) (layers F.Cu B.Cu) (net 2))
+  (via (at 130.5 91.5) (size 0.7) (drill 0.3) (layers F.Cu B.Cu) (net 2))
+  (via (at 136 95.5) (size 0.7) (drill 0.3) (layers F.Cu B.Cu) (net 2))
+  (via (at 169.75 81) (size 0.7) (drill 0.3) (layers F.Cu B.Cu) (net 2))
+  (via (at 170.75 78) (size 0.7) (drill 0.3) (layers F.Cu B.Cu) (net 2))
+  (via (at 165.5 75.75) (size 0.7) (drill 0.3) (layers F.Cu B.Cu) (net 2))
+  (via (at 168 78.5) (size 0.7) (drill 0.3) (layers F.Cu B.Cu) (net 2))
+  (via (at 154 80.25) (size 0.7) (drill 0.3) (layers F.Cu B.Cu) (net 2))
+  (via (at 149.75 78.75) (size 0.7) (drill 0.3) (layers F.Cu B.Cu) (net 2))
+  (via (at 150.25 74.75) (size 0.7) (drill 0.3) (layers F.Cu B.Cu) (net 2))
+  (via (at 153.5 65) (size 0.7) (drill 0.3) (layers F.Cu B.Cu) (net 2))
+  (via (at 154.25 71.25) (size 0.7) (drill 0.3) (layers F.Cu B.Cu) (net 2))
+  (via (at 147.75 67.75) (size 0.7) (drill 0.3) (layers F.Cu B.Cu) (net 2))
+  (via (at 147.5 61.75) (size 0.7) (drill 0.3) (layers F.Cu B.Cu) (net 2))
+  (via (at 135.25 60.75) (size 0.7) (drill 0.3) (layers F.Cu B.Cu) (net 2))
+  (via (at 134.75 67) (size 0.7) (drill 0.3) (layers F.Cu B.Cu) (net 2))
+  (via (at 143.75 72) (size 0.7) (drill 0.3) (layers F.Cu B.Cu) (net 2))
+  (via (at 173 73.5) (size 0.7) (drill 0.3) (layers F.Cu B.Cu) (net 2))
+  (via (at 160.5 62) (size 0.7) (drill 0.3) (layers F.Cu B.Cu) (net 2))
+  (via (at 115.75 76) (size 0.7) (drill 0.3) (layers F.Cu B.Cu) (net 2))
+  (via (at 115.75 72.5) (size 0.7) (drill 0.3) (layers F.Cu B.Cu) (net 2))
+  (via (at 115.75 69) (size 0.7) (drill 0.3) (layers F.Cu B.Cu) (net 2))
+  (via (at 122.5 70.75) (size 0.7) (drill 0.3) (layers F.Cu B.Cu) (net 2))
+  (via (at 125.5 74.5) (size 0.7) (drill 0.3) (layers F.Cu B.Cu) (net 2))
+  (via (at 122.25 81.5) (size 0.7) (drill 0.3) (layers F.Cu B.Cu) (net 2))
+  (via (at 132.75 72.5) (size 0.7) (drill 0.3) (layers F.Cu B.Cu) (net 2))
+  (via (at 128.75 64.25) (size 0.7) (drill 0.3) (layers F.Cu B.Cu) (net 2))
   (segment (start 128.613589 118.25) (end 129.625 118.25) (width 0.25) (layer F.Cu) (net 7))
   (segment (start 124.549989 110.299989) (end 124.549989 114.1864) (width 0.25) (layer F.Cu) (net 7))
@@
       )
     )
+  )
+  (zone (net 2) (net_name GND) (layer F.Cu) (hatch edge 0.508)
+    (connect_pads yes (clearance 0.3))
+    (min_thickness 0.254)
+    (fill yes (arc_segments 16) (thermal_gap 0.508) (thermal_bridge_width 0.508))
+    (polygon
+      (pts
+        (xy 115.25 55.25) (xy 174.75 55.25) (xy 174.75 120.75) (xy 115.25 120.75)
+      )
+    )
+  )
+  (zone (net 2) (net_name GND) (layer B.Cu) (hatch edge 0.508)
+    (connect_pads yes (clearance 0.3))
+    (min_thickness 0.254)
+    (fill yes (arc_segments 16) (thermal_gap 0.508) (thermal_bridge_width 0.508))
+    (polygon
+      (pts
+        (xy 115.25 55.25) (xy 174.75 55.25) (xy 174.75 120.75) (xy 115.25 120.75)
+      )
+    )

Commit message: PCB HW update
Parts:
- added G***: LOGO, kicad:flower, F.Cu at (143.5, 90.8)
- added REF**: OSHW-Logo2_7.3x6mm_SilkScreen, Symbol:OSHW-Logo2_7.3x6mm_SilkScreen, F.Cu at (156.8, 110.0)
- added REF**: Symbol_Barrel_Polarity, Symbol:Symbol_Barrel_Polarity, F.Cu at (166.2, 110.0)
Routing:
- net GND: vias 72 -> 83
